File: board/board.kicad_pcb (KiCad board)
At the start: 2 copper layers, 21 x 13 mm, 1 part

Commit message: initial
Parts:
- added C1: 100nF, Capacitor_SMD:C_0603_1608Metric, F.Cu at (153.6, 112.5)
- added J1: 001_I2C, on_edge:on_edge_2x05_device, F.Cu at (140.0, 96.5)
- added J2: 007_ADC, on_edge:on_edge_2x05_host, F.Cu at (161.0, 128.5)
- added J3: 001_I2C, on_edge:on_edge_2x05_host, F.Cu at (161.0, 96.5)
- added J4: 007_ADC, on_edge:on_edge_2x05_host, F.Cu at (161.0, 112.5)
- added R1: d.n.p, Resistor_SMD:R_0603_1608Metric, F.Cu at (142.9, 112.1)
- added R2: 0R, Resistor_SMD:R_0603_1608Metric, F.Cu at (142.9, 115.1)
- added R3: 0R, Resistor_SMD:R_0603_1608Metric, F.Cu at (152.0, 109.1)
- added R4: d.n.p, Resistor_SMD:R_0603_1608Metric, F.Cu at (153.6, 109.1)
- added R5: d.n.p, Resistor_SMD:R_0603_1608Metric, F.Cu at (144.4, 112.1)
- added R6: 0R, Resistor_SMD:R_0603_1608Metric, F.Cu at (144.4, 115.1)
- added U1: MCP3428, Package_SO:SOIC-14_3.9x8.7mm_P1.27mm, F.Cu at (149.0, 115.5)
- moved LOGO1 32.0 mm to (150.0, 131.0)
Routing:
- net GND: track 0.00 -> 71.4 mm, vias 0 -> 4
- net /5V: track 0.00 -> 60.8 mm, vias 0 -> 4
- net /3.3V: track 0.00 -> 57.6 mm, vias 0 -> 2
- net /adc/SDA: track 0.00 -> 35.9 mm, vias 0 -> 2
- net /adc/SCL: track 0.00 -> 33.0 mm, vias 0 -> 3
- net /adc/AD4+: track 0.00 -> 21.1 mm
- net /adc/AD3-: track 0.00 -> 20.2 mm
- net /adc/AD3+: track 0.00 -> 18.8 mm
- net Net-(J1-Pad5): track 0.00 -> 17.1 mm, vias 0 -> 2
- net Net-(J1-Pad4): track 0.00 -> 16.8 mm, vias 0 -> 2
- net (no net): track 0.00 -> 16.6 mm
- net Net-(J1-Pad8): track 0.00 -> 16.5 mm
- net /adc/AD4-: track 0.00 -> 16.0 mm, vias 0 -> 1
- net Net-(C1-Pad1): track 0.00 -> 15.3 mm
- net /adc/AD2-: track 0.00 -> 12.3 mm, vias 0 -> 1
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Other:
- board size 21 x 13 mm -> 21 x 45 mm
- board text added: "osf.001"
- board text added: "osf.007"
- board text added: "osf.b081.v1.0"
