File: board/board.kicad_sch (KiCad schematic)
At the start: 1 part

Commit message: initial
Parts:
- added J1: 001_I2C, on_edge:on_edge_2x05_device, symbol put_on_edge:001_I2C
- added J2, J4: 007_ADC, on_edge:on_edge_2x05_host, symbol put_on_edge:007_ADC
- added J3: 001_I2C, on_edge:on_edge_2x05_host, symbol put_on_edge:001_I2C
Connections:
- new net: J1.4 (CS/EN), J3.4 (CS/EN)
- new net: J1.5 (INT), J3.5 (INT)
- new net: J1.8 (~{RESET}), J3.8 (~{RESET})
- new net 3.3V: J1.9 (3.3V), J2.9 (3.3V), J3.9 (3.3V), J4.9 (3.3V)
- new net 5V: J1.10 (5V), J2.10 (5V), J3.10 (5V), J4.10 (5V)
- new net GND: J1.1 (GND), J2.1 (GND), J3.1 (GND), J4.1 (GND)
- new net adc/AD1+: J4.3 (ADC0)
- new net adc/AD1-: J4.4 (ADC1)
- new net adc/AD2+: J4.5 (ADC2)
- new net adc/AD2-: J4.6 (ADC3)
- new net adc/AD3+: J2.3 (ADC0)
- new net adc/AD3-: J2.4 (ADC1)
- new net adc/AD4+: J2.5 (ADC2)
- new net adc/AD4-: J2.6 (ADC3)
- new net adc/SCL: J1.3 (SCL), J3.3 (SCL)
- new net adc/SDA: J1.2 (SDA), J3.2 (SDA)
- no-connect marks 0 -> 2
Other:
- sheet implementation renamed adc
- sheet adc: file implementation.kicad_sch -> adc.kicad_sch
- sheet adc ports: added 3.3V, 5V, AD1+, AD1-, AD2+, AD2-, AD3+, AD3-, AD4+, AD4-, GND, SCL, SDA; removed none
- note removed: "Input connectors go here"
- note removed: "Output connectors go here"
